Commit message: Add robo1

File: robo1.urdf (robot description, URDF)
Before this commit: robot flexible, 3 links, 2 joints
Links:
- added link base_link; collision box size=.22 .22 .12; visual box size=.66 .56 .12
- added link body2; collision box size=.22 .22 .12; visual box size=.22 .22 .12
- added link body3; collision box size=.22 .22 .12; visual box size=.22 .22 .12
- added link body4; collision box size=.22 .22 .12; visual box size=.22 .22 .12
- added link cylinder2; collision cylinder length=0.09 radius=0.05; visual cylinder length=0.09 radius=0.05
- added link cylinder3; collision cylinder length=0.09 radius=0.05; visual cylinder length=0.09 radius=0.05
- added link cylinder4; collision cylinder length=0.09 radius=0.05; visual cylinder length=0.09 radius=0.05
- added link leg2; collision box size=.42 .05 .02; visual box size=.42 .05 .02
- added link leg3; collision box size=.42 .05 .02; visual box size=.42 .05 .02
- added link leg4; collision box size=.42 .05 .02; visual box size=.42 .05 .02
- link leg1: geometry collision box size=.42 .05 .02; visual box size=.42 .05 .02
Joints:
- added joint body1_joint: type fixed, parent base_link, child body1
- added joint body2_joint: type fixed, parent base_link, child body2
- added joint body3_joint: type fixed, parent base_link, child body3
- added joint body4_joint: type fixed, parent base_link, child body4
- added joint ignore_cylinder2_joint: type fixed, parent body2, child cylinder2
- added joint ignore_cylinder3_joint: type fixed, parent body3, child cylinder3
- added joint ignore_cylinder4_joint: type fixed, parent body4, child cylinder4
- added joint leg2_joint: type revolute, parent cylinder2, child leg2, origin xyz=0 0.44 -0.06 rpy=0 0 0, axis 1 0 0, limit lower=-1.05 upper=1.05 effort=10 velocity=3
- added joint leg3_joint: type revolute, parent cylinder3, child leg3, origin xyz=0 0 -0.06 rpy=0 0 0, axis 1 0 0, limit lower=-1.05 upper=1.05 effort=10 velocity=3
- added joint leg4_joint: type revolute, parent cylinder4, child leg4, origin xyz=0 0.44 -0.06 rpy=0 0 0, axis 1 0 0, limit lower=-1.05 upper=1.05 effort=10 velocity=3
- joint ignore_cylinder1_joint: origin xyz=0 0.0 0.0 rpy=0 0 0 -> (none)
- joint leg1_joint: origin xyz=0 0.06 0.0 rpy=0 0 0 -> xyz=0 0 -0.06 rpy=0 0 0
